File: hw/pcb/kroneum.kicad_pcb (KiCad board)
At the start: 2 copper layers, 22 parts, among them J1 USB_B_Micro, SW1 Boot_Mode_Btn, SW2 Ctrl_One_Btn, SW3 Reset_Btn, SW4 Ctrl_Ten_Btn, U1 STM32F042F4Px, Y1 16 Mhz

Commit message: hw: switch `ten-1` button from PA5 to PA0 to be able to wake up device from stand-by mode.
Parts:
- R1: value 1k -> 470
Connections:
- U1 pad 12: Ctrl_One -> Net-(U1-Pad12)
- U1 pad 6: Net-(U1-Pad6) -> Ctrl_One
Changed lines of the file:
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@@
   (net 14 "Net-(R2-Pad1)")
   (net 15 BOOT0)
-  (net 16 "Net-(U1-Pad6)")
-  (net 17 "Net-(U1-Pad7)")
-  (net 18 "Net-(U1-Pad8)")
-  (net 19 "Net-(U1-Pad9)")
-  (net 20 "Net-(U1-Pad10)")
-  (net 21 "Net-(U1-Pad14)")
-  (net 22 "Net-(U1-Pad19)")
-  (net 23 "Net-(U1-Pad20)")
-  (net 24 "Net-(BT1-Pad1)")
-  (net 25 "Net-(D1-Pad1)")
-  (net 26 USB_VBUS)
+  (net 16 "Net-(U1-Pad7)")
+  (net 17 "Net-(U1-Pad8)")
+  (net 18 "Net-(U1-Pad9)")
+  (net 19 "Net-(U1-Pad10)")
+  (net 20 "Net-(U1-Pad14)")
+  (net 21 "Net-(U1-Pad19)")
+  (net 22 "Net-(U1-Pad20)")
+  (net 23 "Net-(BT1-Pad1)")
+  (net 24 "Net-(D1-Pad1)")
+  (net 25 USB_VBUS)
+  (net 26 "Net-(U1-Pad12)")
   (net_class Default "This is the default net class."
     (clearance 0.2)
@@
     (add_net "Net-(R2-Pad1)")
     (add_net "Net-(U1-Pad10)")
+    (add_net "Net-(U1-Pad12)")
     (add_net "Net-(U1-Pad14)")
     (add_net "Net-(U1-Pad19)")
     (add_net "Net-(U1-Pad20)")
-    (add_net "Net-(U1-Pad6)")
     (add_net "Net-(U1-Pad7)")
     (add_net "Net-(U1-Pad8)")
@@
       (net 10 USB_D-))
     (pad 1 smd rect (at -1.3 -1.4625) (size 0.4 1.35) (layers F.Cu F.Paste F.Mask)
-      (net 26 USB_VBUS))
+      (net 25 USB_VBUS))
     (pad 5 smd rect (at 1.3 -1.4625) (size 0.4 1.35) (layers F.Cu F.Paste F.Mask)
       (net 1 GND))
@@
       (effects (font (size 1 1) (thickness 0.15)))
     )
-    (fp_text value 1k (at 0 1.65) (layer F.Fab)
+    (fp_text value 470 (at 0 1.65) (layer F.Fab)
       (effects (font (size 1 1) (thickness 0.15)))
     )
@@
       (net 3 VDD))
     (pad 6 smd rect (at -2.95 0.325) (size 1.45 0.45) (layers F.Cu F.Paste F.Mask)
-      (net 16 "Net-(U1-Pad6)"))
+      (net 7 Ctrl_One))
     (pad 7 smd rect (at -2.95 0.975) (size 1.45 0.45) (layers F.Cu F.Paste F.Mask)
-      (net 17 "Net-(U1-Pad7)"))
+      (net 16 "Net-(U1-Pad7)"))
     (pad 8 smd rect (at -2.95 1.625) (size 1.45 0.45) (layers F.Cu F.Paste F.Mask)
-      (net 18 "Net-(U1-Pad8)"))
+      (net 17 "Net-(U1-Pad8)"))
     (pad 9 smd rect (at -2.95 2.275) (size 1.45 0.45) (layers F.Cu F.Paste F.Mask)
-      (net 19 "Net-(U1-Pad9)"))
+      (net 18 "Net-(U1-Pad9)"))
     (pad 10 smd rect (at -2.95 2.925) (size 1.45 0.45) (layers F.Cu F.Paste F.Mask)
-      (net 20 "Net-(U1-Pad10)"))
+      (net 19 "Net-(U1-Pad10)"))
     (pad 11 smd rect (at 2.95 2.925) (size 1.45 0.45) (layers F.Cu F.Paste F.Mask)
       (net 8 Ctrl_Ten))
     (pad 12 smd rect (at 2.95 2.275) (size 1.45 0.45) (layers F.Cu F.Paste F.Mask)
-      (net 7 Ctrl_One))
+      (net 26 "Net-(U1-Pad12)"))
     (pad 13 smd rect (at 2.95 1.625) (size 1.45 0.45) (layers F.Cu F.Paste F.Mask)
       (net 13 Buzzer))
     (pad 14 smd rect (at 2.95 0.975) (size 1.45 0.45) (layers F.Cu F.Paste F.Mask)
-      (net 21 "Net-(U1-Pad14)"))
+      (net 20 "Net-(U1-Pad14)"))
     (pad 15 smd rect (at 2.95 0.325) (size 1.45 0.45) (layers F.Cu F.Paste F.Mask)
       (net 1 GND))
@@
       (net 12 USB_D+))
     (pad 19 smd rect (at 2.95 -2.275) (size 1.45 0.45) (layers F.Cu F.Paste F.Mask)
-      (net 22 "Net-(U1-Pad19)"))
+      (net 21 "Net-(U1-Pad19)"))
     (pad 20 smd rect (at 2.95 -2.925) (size 1.45 0.45) (layers F.Cu F.Paste F.Mask)
-      (net 23 "Net-(U1-Pad20)"))
+      (net 22 "Net-(U1-Pad20)"))
     (model ${KISYS3DMOD}/Package_SO.3dshapes/TSSOP-20_4.4x6.5mm_P0.65mm.wrl
       (at (xyz 0 0 0))
@@
       (net 1 GND))
     (pad 1 thru_hole rect (at 0 0) (size 3 3) (drill 1.5) (layers *.Cu *.Mask)
-      (net 24 "Net-(BT1-Pad1)"))
+      (net 23 "Net-(BT1-Pad1)"))
     (model ${KISYS3DMOD}/Battery.3dshapes/BatteryHolder_Keystone_103_1x20mm.wrl
       (at (xyz 0 0 0))
@@
     (fp_line (start 0.76 1.58) (end -0.7 1.58) (layer F.SilkS) (width 0.12))
     (pad 1 smd rect (at -1 -0.95) (size 0.9 0.8) (layers F.Cu F.Paste F.Mask)
-      (net 25 "Net-(D1-Pad1)"))
+      (net 24 "Net-(D1-Pad1)"))
     (pad 2 smd rect (at -1 0.95) (size 0.9 0.8) (layers F.Cu F.Paste F.Mask)
-      (net 24 "Net-(BT1-Pad1)"))
+      (net 23 "Net-(BT1-Pad1)"))
     (pad 3 smd rect (at 1 0) (size 0.9 0.8) (layers F.Cu F.Paste F.Mask)
       (net 3 VDD))
@@
     (fp_line (start -2.48 2.55) (end -2.48 -2.55) (layer F.CrtYd) (width 0.05))
     (pad 2 smd trapezoid (at 2.667 0 270) (size 1.6 0.85) (rect_delta 0 0.6 ) (layers F.Cu F.Paste F.Mask)
-      (net 26 USB_VBUS))
+      (net 25 USB_VBUS))
     (pad 1 smd rect (at -1.48 -1.5 270) (size 1 1.5) (layers F.Cu F.Paste F.Mask)
       (net 1 GND))
     (pad 2 smd rect (at -1.3335 0 270) (size 1 1.8) (layers F.Cu F.Paste F.Mask)
-      (net 26 USB_VBUS))
+      (net 25 USB_VBUS))
     (pad 3 smd rect (at -1.48 1.5 270) (size 1 1.5) (layers F.Cu F.Paste F.Mask)
-      (net 25 "Net-(D1-Pad1)"))
+      (net 24 "Net-(D1-Pad1)"))
     (pad 2 smd rect (at 1.3335 0 270) (size 2.2 1.84) (layers F.Cu F.Paste F.Mask)
-      (net 26 USB_VBUS))
+      (net 25 USB_VBUS))
     (pad 2 smd trapezoid (at -0.0762 0 90) (size 1.5 1) (rect_delta 0 0.7 ) (layers F.Cu F.Paste F.Mask)
-      (net 26 USB_VBUS))
+      (net 25 USB_VBUS))
     (model ${KISYS3DMOD}/Package_TO_SOT_SMD.3dshapes/SOT-89-3.wrl
       (at (xyz 0 0 0))

Commit message: hw: connect x-button to PA2 instead of PA5 (to have access to wkup4).
Connections:
- U1 pad 11: Ctrl_Ten -> Net-(U1-Pad11)
- U1 pad 8: Net-(U1-Pad8) -> Ctrl_Ten
Changed lines of the file:
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@@
   (net 15 BOOT0)
   (net 16 "Net-(U1-Pad7)")
-  (net 17 "Net-(U1-Pad8)")
-  (net 18 "Net-(U1-Pad9)")
-  (net 19 "Net-(U1-Pad10)")
-  (net 20 "Net-(U1-Pad14)")
-  (net 21 "Net-(U1-Pad19)")
-  (net 22 "Net-(U1-Pad20)")
-  (net 23 "Net-(BT1-Pad1)")
-  (net 24 "Net-(D1-Pad1)")
-  (net 25 USB_VBUS)
-  (net 26 "Net-(U1-Pad12)")
+  (net 17 "Net-(U1-Pad9)")
+  (net 18 "Net-(U1-Pad10)")
+  (net 19 "Net-(U1-Pad14)")
+  (net 20 "Net-(U1-Pad19)")
+  (net 21 "Net-(U1-Pad20)")
+  (net 22 "Net-(BT1-Pad1)")
+  (net 23 "Net-(D1-Pad1)")
+  (net 24 USB_VBUS)
+  (net 25 "Net-(U1-Pad12)")
+  (net 26 "Net-(U1-Pad11)")
   (net_class Default "This is the default net class."
     (clearance 0.2)
@@
     (add_net "Net-(R2-Pad1)")
     (add_net "Net-(U1-Pad10)")
+    (add_net "Net-(U1-Pad11)")
     (add_net "Net-(U1-Pad12)")
     (add_net "Net-(U1-Pad14)")
@@
     (add_net "Net-(U1-Pad20)")
     (add_net "Net-(U1-Pad7)")
-    (add_net "Net-(U1-Pad8)")
     (add_net "Net-(U1-Pad9)")
     (add_net OSC_IN)
@@
       (net 10 USB_D-))
     (pad 1 smd rect (at -1.3 -1.4625) (size 0.4 1.35) (layers F.Cu F.Paste F.Mask)
-      (net 25 USB_VBUS))
+      (net 24 USB_VBUS))
     (pad 5 smd rect (at 1.3 -1.4625) (size 0.4 1.35) (layers F.Cu F.Paste F.Mask)
       (net 1 GND))
@@
       (net 16 "Net-(U1-Pad7)"))
     (pad 8 smd rect (at -2.95 1.625) (size 1.45 0.45) (layers F.Cu F.Paste F.Mask)
-      (net 17 "Net-(U1-Pad8)"))
+      (net 8 Ctrl_Ten))
     (pad 9 smd rect (at -2.95 2.275) (size 1.45 0.45) (layers F.Cu F.Paste F.Mask)
-      (net 18 "Net-(U1-Pad9)"))
+      (net 17 "Net-(U1-Pad9)"))
     (pad 10 smd rect (at -2.95 2.925) (size 1.45 0.45) (layers F.Cu F.Paste F.Mask)
-      (net 19 "Net-(U1-Pad10)"))
+      (net 18 "Net-(U1-Pad10)"))
     (pad 11 smd rect (at 2.95 2.925) (size 1.45 0.45) (layers F.Cu F.Paste F.Mask)
-      (net 8 Ctrl_Ten))
+      (net 26 "Net-(U1-Pad11)"))
     (pad 12 smd rect (at 2.95 2.275) (size 1.45 0.45) (layers F.Cu F.Paste F.Mask)
-      (net 26 "Net-(U1-Pad12)"))
+      (net 25 "Net-(U1-Pad12)"))
     (pad 13 smd rect (at 2.95 1.625) (size 1.45 0.45) (layers F.Cu F.Paste F.Mask)
       (net 13 Buzzer))
     (pad 14 smd rect (at 2.95 0.975) (size 1.45 0.45) (layers F.Cu F.Paste F.Mask)
-      (net 20 "Net-(U1-Pad14)"))
+      (net 19 "Net-(U1-Pad14)"))
     (pad 15 smd rect (at 2.95 0.325) (size 1.45 0.45) (layers F.Cu F.Paste F.Mask)
       (net 1 GND))
@@
       (net 12 USB_D+))
     (pad 19 smd rect (at 2.95 -2.275) (size 1.45 0.45) (layers F.Cu F.Paste F.Mask)
-      (net 21 "Net-(U1-Pad19)"))
+      (net 20 "Net-(U1-Pad19)"))
     (pad 20 smd rect (at 2.95 -2.925) (size 1.45 0.45) (layers F.Cu F.Paste F.Mask)
-      (net 22 "Net-(U1-Pad20)"))
+      (net 21 "Net-(U1-Pad20)"))
     (model ${KISYS3DMOD}/Package_SO.3dshapes/TSSOP-20_4.4x6.5mm_P0.65mm.wrl
       (at (xyz 0 0 0))
@@
       (net 1 GND))
     (pad 1 thru_hole rect (at 0 0) (size 3 3) (drill 1.5) (layers *.Cu *.Mask)
-      (net 23 "Net-(BT1-Pad1)"))
+      (net 22 "Net-(BT1-Pad1)"))
     (model ${KISYS3DMOD}/Battery.3dshapes/BatteryHolder_Keystone_103_1x20mm.wrl
       (at (xyz 0 0 0))
@@
     (fp_line (start 0.76 1.58) (end -0.7 1.58) (layer F.SilkS) (width 0.12))
     (pad 1 smd rect (at -1 -0.95) (size 0.9 0.8) (layers F.Cu F.Paste F.Mask)
-      (net 24 "Net-(D1-Pad1)"))
+      (net 23 "Net-(D1-Pad1)"))
     (pad 2 smd rect (at -1 0.95) (size 0.9 0.8) (layers F.Cu F.Paste F.Mask)
-      (net 23 "Net-(BT1-Pad1)"))
+      (net 22 "Net-(BT1-Pad1)"))
     (pad 3 smd rect (at 1 0) (size 0.9 0.8) (layers F.Cu F.Paste F.Mask)
       (net 3 VDD))
@@
     (fp_line (start -2.48 2.55) (end -2.48 -2.55) (layer F.CrtYd) (width 0.05))
     (pad 2 smd trapezoid (at 2.667 0 270) (size 1.6 0.85) (rect_delta 0 0.6 ) (layers F.Cu F.Paste F.Mask)
-      (net 25 USB_VBUS))
+      (net 24 USB_VBUS))
     (pad 1 smd rect (at -1.48 -1.5 270) (size 1 1.5) (layers F.Cu F.Paste F.Mask)
       (net 1 GND))
     (pad 2 smd rect (at -1.3335 0 270) (size 1 1.8) (layers F.Cu F.Paste F.Mask)
-      (net 25 USB_VBUS))
+      (net 24 USB_VBUS))
     (pad 3 smd rect (at -1.48 1.5 270) (size 1 1.5) (layers F.Cu F.Paste F.Mask)
-      (net 24 "Net-(D1-Pad1)"))
+      (net 23 "Net-(D1-Pad1)"))
     (pad 2 smd rect (at 1.3335 0 270) (size 2.2 1.84) (layers F.Cu F.Paste F.Mask)
-      (net 25 USB_VBUS))
+      (net 24 USB_VBUS))
     (pad 2 smd trapezoid (at -0.0762 0 90) (size 1.5 1) (rect_delta 0 0.7 ) (layers F.Cu F.Paste F.Mask)
-      (net 25 USB_VBUS))
+      (net 24 USB_VBUS))
     (model ${KISYS3DMOD}/Package_TO_SOT_SMD.3dshapes/SOT-89-3.wrl
       (at (xyz 0 0 0))

Commit message: hw: use default pull-downs for PA0 and PA2.
Connections:
- C8 pad 1: GND -> VDD
- C9 pad 1: GND -> VDD
- SW2 pad 2: GND -> VDD
- SW4 pad 2: GND -> VDD
Changed lines of the file:
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@@
     )
     (pad 1 smd roundrect (at -1.025 0) (size 1.15 1.4) (layers F.Cu F.Paste F.Mask) (roundrect_rratio 0.217391)
-      (net 1 GND))
+      (net 3 VDD))
     (pad 2 smd roundrect (at 1.025 0) (size 1.15 1.4) (layers F.Cu F.Paste F.Mask) (roundrect_rratio 0.217391)
       (net 7 Ctrl_One))
@@
       (net 8 Ctrl_Ten))
     (pad 1 smd roundrect (at -1.025 0) (size 1.15 1.4) (layers F.Cu F.Paste F.Mask) (roundrect_rratio 0.217391)
-      (net 1 GND))
+      (net 3 VDD))
     (model ${KISYS3DMOD}/Capacitor_SMD.3dshapes/C_0805_2012Metric.wrl
       (at (xyz 0 0 0))
@@
     )
     (pad 2 smd rect (at 3.98 2.25) (size 1.55 1.3) (layers F.Cu F.Paste F.Mask)
-      (net 1 GND))
+      (net 3 VDD))
     (pad 1 smd rect (at 3.98 -2.25) (size 1.55 1.3) (layers F.Cu F.Paste F.Mask)
       (net 7 Ctrl_One))
@@
       (net 7 Ctrl_One))
     (pad 2 smd rect (at -3.98 2.25) (size 1.55 1.3) (layers F.Cu F.Paste F.Mask)
-      (net 1 GND))
+      (net 3 VDD))
     (model ${KISYS3DMOD}/Button_Switch_SMD.3dshapes/SW_SPST_PTS645.wrl
       (at (xyz 0 0 0))
@@
     (fp_circle (center 0 0) (end 1.75 -0.05) (layer F.Fab) (width 0.1))
     (pad 2 smd rect (at -3.98 2.25) (size 1.55 1.3) (layers F.Cu F.Paste F.Mask)
-      (net 1 GND))
+      (net 3 VDD))
     (pad 1 smd rect (at -3.98 -2.25) (size 1.55 1.3) (layers F.Cu F.Paste F.Mask)
       (net 8 Ctrl_Ten))
@@
       (net 8 Ctrl_Ten))
     (pad 2 smd rect (at 3.98 2.25) (size 1.55 1.3) (layers F.Cu F.Paste F.Mask)
-      (net 1 GND))
+      (net 3 VDD))
     (model ${KISYS3DMOD}/Button_Switch_SMD.3dshapes/SW_SPST_PTS645.wrl
       (at (xyz 0 0 0))
