File: hw/pcb/Rev 0.2/kroneum.kicad_pcb (KiCad board)
At the start: 2 copper layers, 50 x 40 mm, 18 parts, among them J1 USB_B_Micro, J2 SWD_I2C_BOOT, SW1 Boot_Mode_Btn, SW2 Ctrl_One_Btn, SW3 Reset_Btn, SW4 Ctrl_Ten_Btn, U1 STM32F042F4Px

Commit message: hw: convert micro-usb PTH to mechanical NPTH. Export STEP model of the device to Autodesk Fusion 360.
Routing:
- net Net-(J1-Pad6): track 0.00 -> 7.00 mm
Other:
- outline, holes or cut-outs redrawn
Changed lines of the file:
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@@
     (thickness 1.6)
     (drawings 4)
-    (tracks 167)
+    (tracks 169)
     (zones 0)
     (modules 18)
-    (nets 25)
+    (nets 26)
   )
   (page A4)
@@
     (pad_to_mask_clearance 0.051)
     (solder_mask_min_width 0.25)
-    (aux_axis_origin 0 0)
+    (aux_axis_origin 171.33 132.98)
     (visible_elements FFFFFF7F)
     (pcbplotparams
@@
   (net 23 SCL)
   (net 24 "Net-(D1-Pad1)")
+  (net 25 "Net-(J1-Pad6)")
   (net_class Default "This is the default net class."
     (clearance 0.2)
@@
     (add_net "Net-(D1-Pad1)")
     (add_net "Net-(J1-Pad4)")
+    (add_net "Net-(J1-Pad6)")
     (add_net "Net-(U1-Pad10)")
     (add_net "Net-(U1-Pad11)")
@@
     (add_net USB_VBUS)
     (add_net VDD)
+  )
+  (module micro_usb:USB_Micro-B_Molex-105017-0001 (layer F.Cu)
+    (at 124.45 105.35 270)
+    (descr http://www.molex.com/pdm_docs/sd/1050170001_sd.pdf)
+    (tags "Micro-USB SMD Typ-B")
+    (attr smd)
+    (fp_text reference J1 (at -2.5 -3.44) (layer F.SilkS)
+      (effects (font (size 1 1) (thickness 0.15)))
+    )
+    (fp_text value USB_B_Micro (at -0.16 4.65 270) (layer F.Fab)
+      (effects (font (size 1 1) (thickness 0.15)))
+    )
+    (fp_text user "PCB Edge" (at 0 2.6875 270) (layer Dwgs.User)
+      (effects (font (size 0.5 0.5) (thickness 0.08)))
+    )
+    (fp_text user %R (at 0 0.8875 270) (layer F.Fab)
+      (effects (font (size 1 1) (thickness 0.15)))
+    )
+    (fp_line (start -4.4 3.64) (end 4.4 3.64) (layer F.CrtYd) (width 0.05))
+    (fp_line (start 4.4 -2.46) (end 4.4 3.64) (layer F.CrtYd) (width 0.05))
+    (fp_line (start -4.4 -2.46) (end 4.4 -2.46) (layer F.CrtYd) (width 0.05))
+    (fp_line (start -4.4 3.64) (end -4.4 -2.46) (layer F.CrtYd) (width 0.05))
+    (fp_line (start -3.9 -1.7625) (end -3.45 -1.7625) (layer F.SilkS) (width 0.12))
+    (fp_line (start -3.9 0.0875) (end -3.9 -1.7625) (layer F.SilkS) (width 0.12))
+    (fp_line (start 3.9 2.6375) (end 3.9 2.3875) (layer F.SilkS) (width 0.12))
+    (fp_line (start 3.75 3.3875) (end 3.75 -1.6125) (layer F.Fab) (width 0.1))
+    (fp_line (start -3 2.689204) (end 3 2.689204) (layer F.Fab) (width 0.1))
+    (fp_line (start -3.75 3.389204) (end 3.75 3.389204) (layer F.Fab) (width 0.1))
+    (fp_line (start -3.75 -1.6125) (end 3.75 -1.6125) (layer F.Fab) (width 0.1))
+    (fp_line (start -3.75 3.3875) (end -3.75 -1.6125) (layer F.Fab) (width 0.1))
+    (fp_line (start -3.9 2.6375) (end -3.9 2.3875) (layer F.SilkS) (width 0.12))
+    (fp_line (start 3.9 0.0875) (end 3.9 -1.7625) (layer F.SilkS) (width 0.12))
+    (fp_line (start 3.9 -1.7625) (end 3.45 -1.7625) (layer F.SilkS) (width 0.12))
+    (fp_line (start -1.7 -2.3125) (end -1.25 -2.3125) (layer F.SilkS) (width 0.12))
+    (fp_line (start -1.7 -2.3125) (end -1.7 -1.8625) (layer F.SilkS) (width 0.12))
+    (fp_line (start -1.3 -1.7125) (end -1.5 -1.9125) (layer F.Fab) (width 0.1))
+    (fp_line (start -1.1 -1.9125) (end -1.3 -1.7125) (layer F.Fab) (width 0.1))
+    (fp_line (start -1.5 -2.1225) (end -1.1 -2.1225) (layer F.Fab) (width 0.1))
+    (fp_line (start -1.5 -2.1225) (end -1.5 -1.9125) (layer F.Fab) (width 0.1))
+    (fp_line (start -1.1 -2.1225) (end -1.1 -1.9125) (layer F.Fab) (width 0.1))
+    (pad "" thru_hole roundrect (at -2.5 -1.4625 270) (size 1 1) (drill 0.85) (layers *.Cu *.Mask) (roundrect_rratio 0.25))
+    (pad 2 smd rect (at -0.65 -1.4625 270) (size 0.4 1.35) (layers F.Cu F.Paste F.Mask)
+      (net 6 USB_D-))
+    (pad 1 smd rect (at -1.3 -1.4625 270) (size 0.4 1.35) (layers F.Cu F.Paste F.Mask)
+      (net 16 USB_VBUS))
+    (pad 5 smd rect (at 1.3 -1.4625 270) (size 0.4 1.35) (layers F.Cu F.Paste F.Mask)
+      (net 1 GND))
+    (pad 4 smd rect (at 0.65 -1.4625 270) (size 0.4 1.35) (layers F.Cu F.Paste F.Mask)
+      (net 7 "Net-(J1-Pad4)"))
+    (pad 3 smd rect (at 0 -1.4625 270) (size 0.4 1.35) (layers F.Cu F.Paste F.Mask)
+      (net 8 USB_D+))
+    (pad "" thru_hole roundrect (at 2.5 -1.4625 270) (size 1 1) (drill 0.85) (layers *.Cu *.Mask) (roundrect_rratio 0.25))
+    (pad 6 thru_hole roundrect (at -3.5 1.2375 90) (size 1.2 1.9) (drill 0.85) (layers *.Cu *.Mask) (roundrect_rratio 0.25)
+      (net 25 "Net-(J1-Pad6)"))
+    (pad 6 thru_hole roundrect (at 3.5 1.2375 270) (size 1.2 1.9) (drill 0.85) (layers *.Cu *.Mask) (roundrect_rratio 0.25)
+      (net 25 "Net-(J1-Pad6)"))
+    (model ${KISYS3DMOD}/Connector_USB.3dshapes/USB_Micro-B_Molex_47346-0001.step
+      (at (xyz 0 0 0))
+      (scale (xyz 1 1 1))
+      (rotate (xyz 0 0 0))
+    )
   )
   (module Package_TO_SOT_SMD:SOT-89-3 (layer F.Cu)
@@
       (net 10 BOOT0))
   )
-  (module micro_usb:USB_Micro-B_Molex-105017-0001 (layer F.Cu)
-    (at 124.45 105.35 270)
-    (descr http://www.molex.com/pdm_docs/sd/1050170001_sd.pdf)
-    (tags "Micro-USB SMD Typ-B")
-    (attr smd)
-    (fp_text reference J1 (at -2.5 -3.44) (layer F.SilkS)
-      (effects (font (size 1 1) (thickness 0.15)))
-    )
-    (fp_text value USB_B_Micro (at -0.16 4.65 270) (layer F.Fab)
-      (effects (font (size 1 1) (thickness 0.15)))
-    )
-    (fp_text user "PCB Edge" (at 0 2.6875 270) (layer Dwgs.User)
-      (effects (font (size 0.5 0.5) (thickness 0.08)))
-    )
-    (fp_text user %R (at 0 0.8875 270) (layer F.Fab)
-      (effects (font (size 1 1) (thickness 0.15)))
-    )
-    (fp_line (start -4.4 3.64) (end 4.4 3.64) (layer F.CrtYd) (width 0.05))
-    (fp_line (start 4.4 -2.46) (end 4.4 3.64) (layer F.CrtYd) (width 0.05))
-    (fp_line (start -4.4 -2.46) (end 4.4 -2.46) (layer F.CrtYd) (width 0.05))
-    (fp_line (start -4.4 3.64) (end -4.4 -2.46) (layer F.CrtYd) (width 0.05))
-    (fp_line (start -3.9 -1.7625) (end -3.45 -1.7625) (layer F.SilkS) (width 0.12))
-    (fp_line (start -3.9 0.0875) (end -3.9 -1.7625) (layer F.SilkS) (width 0.12))
-    (fp_line (start 3.9 2.6375) (end 3.9 2.3875) (layer F.SilkS) (width 0.12))
-    (fp_line (start 3.75 3.3875) (end 3.75 -1.6125) (layer F.Fab) (width 0.1))
-    (fp_line (start -3 2.689204) (end 3 2.689204) (layer F.Fab) (width 0.1))
-    (fp_line (start -3.75 3.389204) (end 3.75 3.389204) (layer F.Fab) (width 0.1))
-    (fp_line (start -3.75 -1.6125) (end 3.75 -1.6125) (layer F.Fab) (width 0.1))
-    (fp_line (start -3.75 3.3875) (end -3.75 -1.6125) (layer F.Fab) (width 0.1))
-    (fp_line (start -3.9 2.6375) (end -3.9 2.3875) (layer F.SilkS) (width 0.12))
-    (fp_line (start 3.9 0.0875) (end 3.9 -1.7625) (layer F.SilkS) (width 0.12))
-    (fp_line (start 3.9 -1.7625) (end 3.45 -1.7625) (layer F.SilkS) (width 0.12))
-    (fp_line (start -1.7 -2.3125) (end -1.25 -2.3125) (layer F.SilkS) (width 0.12))
-    (fp_line (start -1.7 -2.3125) (end -1.7 -1.8625) (layer F.SilkS) (width 0.12))
-    (fp_line (start -1.3 -1.7125) (end -1.5 -1.9125) (layer F.Fab) (width 0.1))
-    (fp_line (start -1.1 -1.9125) (end -1.3 -1.7125) (layer F.Fab) (width 0.1))
-    (fp_line (start -1.5 -2.1225) (end -1.1 -2.1225) (layer F.Fab) (width 0.1))
-    (fp_line (start -1.5 -2.1225) (end -1.5 -1.9125) (layer F.Fab) (width 0.1))
-    (fp_line (start -1.1 -2.1225) (end -1.1 -1.9125) (layer F.Fab) (width 0.1))
-    (pad "" thru_hole roundrect (at -2.5 -1.4625 270) (size 1.45 1.45) (drill 0.85) (layers *.Cu *.Mask) (roundrect_rratio 0.25))
-    (pad 2 smd rect (at -0.65 -1.4625 270) (size 0.4 1.35) (layers F.Cu F.Paste F.Mask)
-      (net 6 USB_D-))
-    (pad 1 smd rect (at -1.3 -1.4625 270) (size 0.4 1.35) (layers F.Cu F.Paste F.Mask)
-      (net 16 USB_VBUS))
-    (pad 5 smd rect (at 1.3 -1.4625 270) (size 0.4 1.35) (layers F.Cu F.Paste F.Mask)
-      (net 1 GND))
-    (pad 4 smd rect (at 0.65 -1.4625 270) (size 0.4 1.35) (layers F.Cu F.Paste F.Mask)
-      (net 7 "Net-(J1-Pad4)"))
-    (pad 3 smd rect (at 0 -1.4625 270) (size 0.4 1.35) (layers F.Cu F.Paste F.Mask)
-      (net 8 USB_D+))
-    (pad "" thru_hole roundrect (at 2.5 -1.4625 270) (size 1.45 1.45) (drill 0.85) (layers *.Cu *.Mask) (roundrect_rratio 0.25))
-    (pad "" thru_hole roundrect (at -3.5 1.2375 90) (size 1.2 1.9) (drill 0.85) (layers *.Cu *.Mask) (roundrect_rratio 0.25))
-    (pad "" thru_hole roundrect (at 3.5 1.2375 270) (size 1.2 1.9) (drill 0.85) (layers *.Cu *.Mask) (roundrect_rratio 0.25))
-    (model ${KISYS3DMOD}/Connector_USB.3dshapes/USB_Micro-B_Molex_47346-0001.step
-      (at (xyz 0 0 0))
-      (scale (xyz 1 1 1))
-      (rotate (xyz 0 0 0))
-    )
-  )
   (gr_line (start 171.35 133) (end 121.35 133) (layer Edge.Cuts) (width 0.15))
   (gr_line (start 171.35 93) (end 171.35 133) (layer Edge.Cuts) (width 0.15))
-  (gr_line (start 121.4 93) (end 171.35 93) (layer Edge.Cuts) (width 0.15))
+  (gr_line (start 121.35 93) (end 171.35 93) (layer Edge.Cuts) (width 0.15))
   (gr_line (start 121.35 133) (end 121.35 93) (layer Edge.Cuts) (width 0.15))
   (segment (start 125.9125 106.65) (end 126.3875 106.65) (width 0.4064) (layer F.Cu) (net 1))
@@
   (segment (start 146.48 111.69) (end 146.48 114) (width 0.4064) (layer F.Cu) (net 23))
   (segment (start 131.17 106.46) (end 131.17 104.34) (width 0.762) (layer F.Cu) (net 24))
+  (segment (start 123.2125 102.55) (end 123.2125 108.85) (width 0.4064) (layer F.Cu) (net 25))
+  (segment (start 123.2125 101.85) (end 123.2125 102.55) (width 0.4064) (layer F.Cu) (net 25))
 )

Commit message: hw: decrease width of TSSOP20 pads, first export of Gerbers.
Parts:
- U1: footprint Package_SO:TSSOP-20_4.4x6.5mm_P0.65mm -> tssop-20x6.5mmx4:TSSOP-20_4.4x6.5mm_P0.65mm

Commit message: hw: add decoupling capacitors for the voltage regulator.
Parts:
- added C2: 10u, Capacitor_SMD:C_0805_2012Metric_Pad1.15x1.40mm_HandSolder, F.Cu at (128.8, 101.5)
- added C4: 10u, Capacitor_SMD:C_0805_2012Metric_Pad1.15x1.40mm_HandSolder, F.Cu at (129.0, 108.5)
- moved D1 2.14 mm to (132.9, 109.4)
Routing:
- net Net-(C4-Pad1): track 2.12 -> 6.56 mm
- net USB_D+: track 22.3 -> 24.8 mm
- net USB_D-: track 21.5 -> 22.8 mm
- net VDD: track 99.9 -> 99.1 mm
