File: hw/pcb/Rev_0.3/kroneum.kicad_pcb (KiCad board)
At the start: 2 copper layers, 43.7 x 40 mm, 23 parts, among them J1 USB_B_Micro, SW1 Boot_Mode_Btn, SW2 Ctrl_One_Btn, SW3 Reset_Btn, SW4 Ctrl_Ten_Btn, U1 STM32F042F4Px

Commit message: hw: finish PCB Rev 0.3
Routing:
- net GND: track 109.3 -> 83.8 mm
- added copper zone on F.Cu, net GND
Changed lines of the file:
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@@
     (thickness 1.6)
     (drawings 4)
-    (tracks 163)
+    (tracks 158)
     (zones 0)
     (modules 23)
@@
   )
   (setup
-    (last_trace_width 0.762)
+    (last_trace_width 0.4064)
     (user_trace_width 0.4064)
     (user_trace_width 0.4572)
@@
     (user_trace_width 1.524)
     (trace_clearance 0.2)
-    (zone_clearance 0.508)
+    (zone_clearance 0.5)
     (zone_45_only no)
     (trace_min 0.25)
@@
   (segment (start 142.875 108.7264) (end 142.875 108.025) (width 0.4064) (layer F.Cu) (net 1))
   (segment (start 145.05 109.77) (end 143.9186 109.77) (width 0.4064) (layer F.Cu) (net 1))
-  (segment (start 143.65 105.1) (end 142.875 105.875) (width 0.762) (layer F.Cu) (net 1))
-  (segment (start 143.65 99.125) (end 143.65 105.1) (width 0.762) (layer F.Cu) (net 1))
   (segment (start 125.9125 101.8) (end 127.05 101.8) (width 0.4064) (layer F.Cu) (net 1))
-  (segment (start 128.007 102.757) (end 128.007 103.608) (width 0.4064) (layer F.Cu) (net 1))
-  (segment (start 127.05 101.8) (end 128.007 102.757) (width 0.4064) (layer F.Cu) (net 1))
   (segment (start 130.885 95.665) (end 131.44 96.22) (width 0.762) (layer F.Cu) (net 1))
   (segment (start 128.81 95.665) (end 130.885 95.665) (width 0.762) (layer F.Cu) (net 1))
   (segment (start 143.65 98.075) (end 143.65 99.125) (width 0.762) (layer F.Cu) (net 1))
-  (segment (start 141.24 95.665) (end 143.65 98.075) (width 0.762) (layer F.Cu) (net 1))
-  (segment (start 132.245 95.665) (end 134.025 95.665) (width 0.762) (layer F.Cu) (net 1))
-  (segment (start 131.69 96.22) (end 132.245 95.665) (width 0.762) (layer F.Cu) (net 1))
   (segment (start 131.44 96.22) (end 131.69 96.22) (width 0.762) (layer F.Cu) (net 1))
-  (segment (start 134.025 95.665) (end 141.24 95.665) (width 0.762) (layer F.Cu) (net 1))
   (segment (start 142.925 105.875) (end 142.925 108.025) (width 0.762) (layer F.Cu) (net 1))
   (segment (start 150.938 99.125) (end 152.35 99.125) (width 0.762) (layer F.Cu) (net 2))
@@
   (segment (start 148.05 115.025) (end 149.425 116.4) (width 0.4064) (layer F.Cu) (net 23))
   (segment (start 148.455 111.72) (end 148.05 112.125) (width 0.4064) (layer F.Cu) (net 23))
-  (segment (start 124.5475 95.665) (end 128.81 95.665) (width 0.762) (layer F.Cu) (net 1))
-  (segment (start 123.2125 97) (end 124.5475 95.665) (width 0.762) (layer F.Cu) (net 1))
   (segment (start 123.2125 97) (end 123.2125 104) (width 0.762) (layer F.Cu) (net 1))
-  (segment (start 125.4125 101.8) (end 123.2125 104) (width 0.4064) (layer F.Cu) (net 1))
-  (segment (start 125.9125 101.8) (end 125.4125 101.8) (width 0.4064) (layer F.Cu) (net 1))
   (segment (start 123.2125 112.3075) (end 130.725 119.82) (width 0.762) (layer F.Cu) (net 1))
   (segment (start 123.2125 104) (end 123.2125 112.3075) (width 0.762) (layer F.Cu) (net 1))
@@
   (segment (start 140.7 121.475) (end 139.045 119.82) (width 0.762) (layer F.Cu) (net 1))
   (segment (start 141.5 121.475) (end 140.7 121.475) (width 0.762) (layer F.Cu) (net 1))
-  (segment (start 142.975 130.025) (end 143.85 130.9) (width 0.762) (layer F.Cu) (net 1))
-  (segment (start 141.5 130.025) (end 142.975 130.025) (width 0.762) (layer F.Cu) (net 1))
   (segment (start 143.85 130.9) (end 150.15 130.9) (width 0.762) (layer F.Cu) (net 1))
   (segment (start 141.5 130.025) (end 137.85 130.025) (width 0.762) (layer F.Cu) (net 1))
   (segment (start 130.725 122.9) (end 130.725 119.82) (width 0.762) (layer F.Cu) (net 1))
   (segment (start 137.85 130.025) (end 130.725 122.9) (width 0.762) (layer F.Cu) (net 1))
+  (segment (start 125.9125 101.8) (end 124.8311 101.8) (width 0.4064) (layer F.Cu) (net 1))
+  (segment (start 142.975 130.025) (end 143.85 130.9) (width 0.762) (layer F.Cu) (net 1))
+  (segment (start 141.5 130.025) (end 142.975 130.025) (width 0.762) (layer F.Cu) (net 1))
+  (segment (start 128.007 102.707) (end 128.007 103.608) (width 0.4064) (layer F.Cu) (net 1))
+  (segment (start 125.9125 101.8) (end 127.1 101.8) (width 0.4064) (layer F.Cu) (net 1))
+  (segment (start 127.1 101.8) (end 128.007 102.707) (width 0.4064) (layer F.Cu) (net 1))
+  (segment (start 146.1814 109.77) (end 146.5264 109.425) (width 0.4064) (layer F.Cu) (net 1))
+  (segment (start 145.05 109.77) (end 146.1814 109.77) (width 0.4064) (layer F.Cu) (net 1))
+  (segment (start 146.5264 109.425) (end 147.2 109.425) (width 0.4064) (layer F.Cu) (net 1))
   (segment (start 158.1 117.85) (end 158.1 124.15) (width 0.762) (layer F.Cu) (net 3))
   (segment (start 161.9 101.85) (end 161.9 108.15) (width 0.762) (layer F.Cu) (net 3))
@@
   (segment (start 131.44 99.22) (end 131.44 101.7) (width 0.762) (layer F.Cu) (net 24))
   (segment (start 131.44 101.7) (end 130.057 103.083) (width 0.762) (layer F.Cu) (net 24))
+  (zone (net 1) (net_name GND) (layer F.Cu) (hatch none 0.508)
+    (connect_pads (clearance 0.5))
+    (min_thickness 0.3)
+    (fill yes (arc_segments 32) (thermal_gap 0.6) (thermal_bridge_width 0.6))
+    (polygon
+      (pts
+        (xy 121.375 93.025) (xy 165 93) (xy 165 133) (xy 121.35 132.975)
+      )
+    )
+    (polygon
+      (pts
+        (xy 126.75 101.1) (xy 128.1 101.125) (xy 128.15 102.925) (xy 126.825 102.95)
+      )
+    )
+    (polygon
+      (pts
+        (xy 126.3 96.15) (xy 127.875 96.25) (xy 127.475 98.75) (xy 125.95 98.7)
+      )
+    )
+    (polygon
+      (pts
+        (xy 139.475 109.15) (xy 141.75 109.15) (xy 141.75 114.475) (xy 139.6 114.475) (xy 139.6 109.2)
+      )
+    )
+  )
 )
